File: elec/layout/default/bno055.kicad_pcb (KiCad board)
At the start: 2 copper layers, 225.7 x 100.8 mm, 0 parts

Commit message: initial design
Parts:
- added C1: Multilayer Ceramic Capacitors MLCC - SMD/SMT 100nF 10V 0402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, lib:C0402, F.Cu at (118.8, 51.2)
- added C2: Multilayer Ceramic Capacitors MLCC - SMD/SMT 1uF 6.3V 0402 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, lib:C0402, F.Cu at (116.9, 51.2)
- added C3: Multilayer Ceramic Capacitors MLCC - SMD/SMT 100nF 10V 0402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, lib:C0402, F.Cu at (121.5, 48.2)
- added C4: Multilayer Ceramic Capacitors MLCC - SMD/SMT 20pF 50V 0402 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, lib:C0402, F.Cu at (113.0, 51.7)
- added C5: Multilayer Ceramic Capacitors MLCC - SMD/SMT 20pF 50V 0402 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, lib:C0402, F.Cu at (113.1, 46.6)
- added R1: Chip Resistor - Surface Mount 10KOhms ±5% 1/16W 0402 RoHS, lib:R0402, F.Cu at (118.8, 44.0)
- added R2: Chip Resistor - Surface Mount 10KOhms ±5% 1/16W 0402 RoHS, lib:R0402, F.Cu at (121.5, 49.3)
- added R3: Chip Resistor - Surface Mount 10KOhms ±5% 1/16W 0402 RoHS, lib:R0402, F.Cu at (121.6, 50.4)
- added U1: , lib:LGA-28_L5.2-W3.8-P0.50-BL, F.Cu at (118.0, 47.6)
- added U2: , lib:FC-135R_L3.2-W1.5, F.Cu at (113.0, 49.1)
Routing:
- net xin32: track 0.00 -> 5.61 mm
- net vcc: track 0.00 -> 5.23 mm
- net xout32: track 0.00 -> 5.04 mm
- net ps1: track 0.00 -> 2.65 mm
- net ps0: track 0.00 -> 1.69 mm
- net cap: track 0.00 -> 1.55 mm
- net com3: track 0.00 -> 1.38 mm
